File: pcb/cad/MBTemp3_Eurocard.kicad_pcb (KiCad board)
At the start: 2 copper layers, 160 x 100 mm, 143 parts, among them J10 RJ25, J3 RJ11, J4 RJ11, J5 RJ11, J6 RJ11, J9 RJ25, K1 Jack, P0 EURO BOARD, P1 Endereço, P2 Programação, P3 CONN_02X10, P4 CONN_1, SW1 -5V, SW2 +6V, U1 74HC4051, U10 REF5050, U11 OPA2277, U12 AD8139, U13 ADS8318, U14 DCR010505U, U15 LT3015, U16 DCP010512D, U17 LT3080, U18 LT3080, U19 LT3015, U2 74HC4051, U3 74HC4051, U4 LT3092, U5 REF5025, U6 IL3685, U7 PIC16F887A_TQFP, U8 LT3582, U9 LT3080, X1 16MHz

Commit message: v2.4
Parts:
- moved REF1 3.00 mm to (72.9, 138.7)
- moved REF3 3.00 mm to (72.9, 52.7)
Other:
- board text added: "MBTemp - 2.4 Junho/2017 Marcelo Bacchetti Bruno V. Luvizotto Patrícia H. Nallin"
- board text removed: "MBTemp - 2.4 Março/2017 Marcelo Bacchetti Bruno V. Luvizotto Patrícia H. Nallin"
Changed lines of the file:
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@@
     (area 58.955379 43.03418 227.99 156.02619)
     (thickness 1.6002)
-    (drawings 68)
+    (drawings 70)
     (tracks 1678)
     (zones 0)
@@
       (drillshape 0)
       (scaleselection 1)
-      (outputdirectory "Gerber_v2-4 28Abril-2017/"))
+      (outputdirectory ../Gerber/))
   )
   (net 0 "")
@@
   )
   (module Mounting_Holes:MountingHole_3.2mm_M3_ISO14580_Pad (layer Superior)
-    (at 69.9412 138.6944)
+    (at 72.9412 138.6944)
     (descr "Mounting Hole 3.2mm, M3, ISO14580")
     (tags "mounting hole 3.2mm m3 iso14580")
@@
   )
   (module Mounting_Holes:MountingHole_3.2mm_M3_ISO14580_Pad (layer Superior)
-    (at 69.9412 52.72)
+    (at 72.9412 52.72)
     (descr "Mounting Hole 3.2mm, M3, ISO14580")
     (tags "mounting hole 3.2mm m3 iso14580")
@@
     (pad 0 thru_hole circle (at -6.78 7.59914 270) (size 2.5 2.5) (drill 1.6) (layers *.Cu *.Mask F.SilkS))
   )
+  (gr_line (start 59.7412 50) (end 59.7412 150) (angle 90) (layer Dwgs.User) (width 0.15))
+  (gr_line (start 61.3412 50) (end 61.3412 150) (angle 90) (layer Dwgs.User) (width 0.15))
   (gr_line (start 226.3862 69.15) (end 226.3862 64) (angle 90) (layer F.SilkS) (width 0.15))
   (gr_text ". . . . . ." (at 84.9 139.9 90) (layer F.SilkS)
@@
     (effects (font (size 1.2 1.2) (thickness 0.2)))
   )
-  (gr_text "MBTemp - 2.4\nMarço/2017\nMarcelo Bacchetti\nBruno V. Luvizotto\nPatrícia H. Nallin" (at 127.125 58.4) (layer F.SilkS)
+  (gr_text "MBTemp - 2.4\nJunho/2017\nMarcelo Bacchetti\nBruno V. Luvizotto\nPatrícia H. Nallin" (at 127.125 58.4) (layer F.SilkS)
     (effects (font (size 2.032 1.524) (thickness 0.2)))
   )
