File: pcb/cad/MBTemp3_Eurocard.sch (KiCad schematic (older format))
At the start: 12 parts, among them J3 RJ11, J4 RJ11, J5 RJ11, J6 RJ11, P3 CONN_02X10, U1 74HC4051, U2 74HC4051, U3 74HC4051, U4 LT3092

Commit message: v2.4
Changed lines of the file:
@@
 LIBS:Pt100-cache
 LIBS:Controle
-LIBS:MBTemp3_Eurocard-cache
 EELAYER 25 0
 EELAYER END
@@
 encoding utf-8
 Sheet 1 4
-Title ""
-Date "28 oct 2014"
-Rev ""
+Title "MBTemp Eurocard"
+Date "2017-06-20"
+Rev "V2.4"
 Comp ""
 Comment1 ""
@@
 PT100_Diff+
 $Sheet
-S 7650 5550 1000 950
+S 7325 5120 1000 950
 U 5087D3F4
 F0 "ADC" 60
@@
 A
 $Sheet
-S 3000 5700 2250 1600
+S 3030 5160 2250 1600
 U 503F7772
 F0 "PIC" 60
@@
 $EndComp
 $Sheet
-S 5650 5750 1300 950
+S 5615 5135 1300 950
 U 50211263
 F0 "Alimentacao" 60

Commit message: v2.5
Parts:
- added C54, C55, C56, C57, C58, C59, C60, C61: 10uF, symbol C_Small
- added R27, R32: 0, symbol R-RESCUE-MBTemp3
Connections:
- net GND: now also C54.2, C55.2, C56.2, C57.2, C58.2, C59.2, C60.2, C61.2, R32.2; no longer U3.6 (Inh)
- net J3_1: now reaches J3.1, U1.15 (X2)
- net J3_1: now also C54.1
- net J3_2: now reaches J3.2, U2.15 (X2)
- net J3_2: now also C55.1
- net J3_4: now reaches J3.4, U3.15 (X2)
- net J4_1: now reaches J4.1, U1.12 (X3)
- net J4_1: now also C56.1
- net J4_2: now reaches J4.2, U2.12 (X3)
- net J4_2: now also C57.1
- net J4_4: now reaches J4.4, U3.12 (X3)
- net J5_1: now reaches J5.1, U1.1 (X4)
- net J5_1: now also C58.1
- net J5_4: now reaches J5.4, U3.1 (X4)
- net J6_1: now reaches J6.1, U1.5 (X5)
- net J6_1: now also C60.1
- net J6_2: now reaches J6.2, U2.5 (X5)
- net J6_2: now also C61.1
- net J6_4: now reaches J6.4, U3.5 (X5)
- net J8_1 renamed J5_2
- net J5_2: now also C59.1
- new net I_EN: R27.1, R32.1, U3.6 (Inh)
- new net I_ENABLE: R27.2
Other:
- moved on the sheet: J3, J4, J5, J6, P3, R1, R2, R3, U1, U2, U3, U4
