File: pcb/cad/Projeto007-Sensor-Temperatura.sch (KiCad schematic (older format))
At the start: 26 parts, among them U10 REF5050, U11 OPA2277, U12 AD8139, U13 ADS8318, U5 REF5025

Commit message: v2.5
Parts:
- C19, C20: value 47pF -> 1uF
Changed lines of the file:
@@
 EESchema Schematic File Version 2
-LIBS:MBTemp3_Eurocard-rescue
-LIBS:MBTemp3-rescue
 LIBS:power
 LIBS:device
@@
 LIBS:contrib
 LIBS:valves
-LIBS:Pt100-cache
-LIBS:Controle
+LIBS:MBTemp3_Eurocard-cache
 EELAYER 25 0
 EELAYER END
@@
 $EndDescr
 $Comp
-L GND-RESCUE-MBTemp3 #PWR013
+L GND-RESCUE-MBTemp3 #PWR017
 U 1 1 514B3706
 P 6300 6450
-F 0 "#PWR013" H 6300 6450 30  0001 C CNN
+F 0 "#PWR017" H 6300 6450 30  0001 C CNN
 F 1 "GND" H 6300 6380 30  0001 C CNN
 F 2 "" H 6300 6450 60  0001 C CNN
@@
 $EndComp
 $Comp
-L GND-RESCUE-MBTemp3 #PWR014
+L GND-RESCUE-MBTemp3 #PWR018
 U 1 1 514B36FC
 P 4700 6450
-F 0 "#PWR014" H 4700 6450 30  0001 C CNN
+F 0 "#PWR018" H 4700 6450 30  0001 C CNN
 F 1 "GND" H 4700 6380 30  0001 C CNN
 F 2 "" H 4700 6450 60  0001 C CNN
@@
 $EndComp
 $Comp
-L GND-RESCUE-MBTemp3 #PWR015
+L GND-RESCUE-MBTemp3 #PWR019
 U 1 1 514B3460
 P 5500 4650
-F 0 "#PWR015" H 5500 4650 30  0001 C CNN
+F 0 "#PWR019" H 5500 4650 30  0001 C CNN
 F 1 "GND" H 5500 4580 30  0001 C CNN
 F 2 "" H 5500 4650 60  0001 C CNN
@@
 AR Path="/5087D3F4/510A8266" Ref="C19"  Part="1"
 F 0 "C19" H 4300 4850 50  0000 L CNN
-F 1 "47pF" H 4250 4650 50  0000 L CNN
+F 1 "1uF" H 4250 4650 50  0000 L CNN
 F 2 "" H 4500 4750 60  0001 C CNN
 F 3 "" H 4500 4750 60  0001 C CNN
@@
 AR Path="/5087D3F4/510A8241" Ref="C20"  Part="1"
 F 0 "C20" H 6400 4850 50  0000 L CNN
-F 1 "47pF" H 6350 4650 50  0000 L CNN
+F 1 "1uF" H 6350 4650 50  0000 L CNN
 F 2 "" H 6600 4750 60  0001 C CNN
 F 3 "" H 6600 4750 60  0001 C CNN
@@
 $EndComp
 $Comp
-L GND-RESCUE-MBTemp3 #PWR016
+L GND-RESCUE-MBTemp3 #PWR020
 U 1 1 510A8149
 P 4950 3700
-F 0 "#PWR016" H 4950 3700 30  0001 C CNN
+F 0 "#PWR020" H 4950 3700 30  0001 C CNN
 F 1 "GND" H 4950 3630 30  0001 C CNN
 F 2 "" H 4950 3700 60  0001 C CNN
@@
 $EndComp
 $Comp
-L +5V #PWR017
+L +5V #PWR021
 U 1 1 5087DBE7
 P 4700 3050
-F 0 "#PWR017" H 4700 3140 20  0001 C CNN
+F 0 "#PWR021" H 4700 3140 20  0001 C CNN
 F 1 "+5V" H 4675 3175 30  0000 C CNN
 F 2 "" H 4700 3050 60  0001 C CNN
@@
 $EndComp
 $Comp
-L GND-RESCUE-MBTemp3 #PWR018
+L GND-RESCUE-MBTemp3 #PWR022
 U 1 1 508195DD
 P 3250 1850
-F 0 "#PWR018" H 3250 1850 30  0001 C CNN
+F 0 "#PWR022" H 3250 1850 30  0001 C CNN
 F 1 "GND" H 3250 1780 30  0001 C CNN
 F 2 "" H 3250 1850 60  0001 C CNN
@@
 $EndComp
 $Comp
-L GND-RESCUE-MBTemp3 #PWR019
+L GND-RESCUE-MBTemp3 #PWR023
 U 1 1 508195D4
 P 2850 2950
-F 0 "#PWR019" H 2850 2950 30  0001 C CNN
+F 0 "#PWR023" H 2850 2950 30  0001 C CNN
 F 1 "GND" H 2850 2880 30  0001 C CNN
 F 2 "" H 2850 2950 60  0001 C CNN
@@
 $EndComp
 $Comp
-L GND-RESCUE-MBTemp3 #PWR020
+L GND-RESCUE-MBTemp3 #PWR024
 U 1 1 508195C8
 P 7300 2700
-F 0 "#PWR020" H 7300 2700 30  0001 C CNN
+F 0 "#PWR024" H 7300 2700 30  0001 C CNN
 F 1 "GND" H 7300 2630 30  0001 C CNN
 F 2 "" H 7300 2700 60  0001 C CNN
@@
 $EndComp
 $Comp
-L GND-RESCUE-MBTemp3 #PWR021
+L GND-RESCUE-MBTemp3 #PWR025
 U 1 1 508195B7
 P 7600 6200
-F 0 "#PWR021" H 7600 6200 30  0001 C CNN
+F 0 "#PWR025" H 7600 6200 30  0001 C CNN
 F 1 "GND" H 7600 6130 30  0001 C CNN
 F 2 "" H 7600 6200 60  0001 C CNN
@@
 $EndComp
 $Comp
-L GND-RESCUE-MBTemp3 #PWR022
+L GND-RESCUE-MBTemp3 #PWR026
 U 1 1 508195AE
 P 2850 6300
-F 0 "#PWR022" H 2850 6300 30  0001 C CNN
+F 0 "#PWR026" H 2850 6300 30  0001 C CNN
 F 1 "GND" H 2850 6230 30  0001 C CNN
 F 2 "" H 2850 6300 60  0001 C CNN
@@
 Connection ~ 7150 3100
 $Comp
-L GND-RESCUE-MBTemp3 #PWR023
+L GND-RESCUE-MBTemp3 #PWR027
 U 1 1 544FC342
 P 7150 3700
-F 0 "#PWR023" H 7150 3700 30  0001 C CNN
+F 0 "#PWR027" H 7150 3700 30  0001 C CNN
 F 1 "GND" H 7150 3630 30  0001 C CNN
 F 2 "" H 7150 3700 60  0001 C CNN
@@
 	7150 3700 7150 3600
 $Comp
-L +6V #PWR024
+L +6V #PWR028
 U 1 1 57DC0E7F
 P 4400 3450
-F 0 "#PWR024" H 4400 3300 50  0001 C CNN
+F 0 "#PWR028" H 4400 3300 50  0001 C CNN
 F 1 "+6V" H 4400 3590 50  0000 C CNN
 F 2 "" H 4400 3450 50  0000 C CNN
@@
 $EndComp
 $Comp
-L +6V #PWR025
+L +6V #PWR029
 U 1 1 57DC0F86
 P 4700 5350
-F 0 "#PWR025" H 4700 5200 50  0001 C CNN
+F 0 "#PWR029" H 4700 5200 50  0001 C CNN
 F 1 "+6V" H 4700 5490 50  0000 C CNN
 F 2 "" H 4700 5350 50  0000 C CNN
@@
 $EndComp
 $Comp
-L +6V #PWR026
+L +6V #PWR030
 U 1 1 57DC10D4
 P 1100 950
-F 0 "#PWR026" H 1100 800 50  0001 C CNN
+F 0 "#PWR030" H 1100 800 50  0001 C CNN
 F 1 "+6V" H 1100 1090 50  0000 C CNN
 F 2 "" H 1100 950 50  0000 C CNN
@@
 $EndComp
 $Comp
-L -5V #PWR25
+L -5V #PWR29
 U 1 1 57DC13EF
 P 6350 5500
-F 0 "#PWR25" H 6350 5600 50  0001 C CNN
+F 0 "#PWR29" H 6350 5600 50  0001 C CNN
 F 1 "-5V" H 6350 5650 50  0000 C CNN
 F 2 "" H 6350 5500 50  0000 C CNN
@@
 $EndComp
 $Comp
-L -5V #PWR16
+L -5V #PWR20
 U 1 1 57DC14C2
 P 2900 4450
-F 0 "#PWR16" H 2900 4550 50  0001 C CNN
+F 0 "#PWR20" H 2900 4550 50  0001 C CNN
 F 1 "-5V" H 2900 4600 50  0000 C CNN
 F 2 "" H 2900 4450 50  0000 C CNN
