File: pcb/cad/Pic.sch (KiCad schematic (older format))
At the start: 36 parts, among them J10 RJ25, J9 RJ25, P1 Endereço, P2 Programação, U14 DCR010505U, U6 IL3685, U7 PIC16F887A_TQFP, X1 16MHz

Commit message: v2.5
Connections:
- net I_ENABLE: now reaches U7.11 (RB3/PGM)
Changed lines of the file:
@@
 EESchema Schematic File Version 2
-LIBS:MBTemp3_Eurocard-rescue
-LIBS:MBTemp3-rescue
 LIBS:power
 LIBS:device
@@
 LIBS:contrib
 LIBS:valves
-LIBS:Pt100-cache
-LIBS:Controle
+LIBS:MBTemp3_Eurocard-cache
 EELAYER 25 0
 EELAYER END
@@
 $EndDescr
 $Comp
-L GND-RESCUE-MBTemp3 #PWR027
+L GND-RESCUE-MBTemp3 #PWR031
 U 1 1 51484804
 P 8950 3350
-F 0 "#PWR027" H 8950 3350 30  0001 C CNN
+F 0 "#PWR031" H 8950 3350 30  0001 C CNN
 F 1 "GND" H 8950 3280 30  0001 C CNN
 F 2 "" H 8950 3350 60  0001 C CNN
@@
 $EndComp
 $Comp
-L +5V #PWR028
+L +5V #PWR032
 U 1 1 509150E6
 P 9300 900
-F 0 "#PWR028" H 9300 990 20  0001 C CNN
+F 0 "#PWR032" H 9300 990 20  0001 C CNN
 F 1 "+5V" H 9300 990 30  0000 C CNN
 F 2 "" H 9300 900 60  0001 C CNN
@@
 A
 $Comp
-L GND-RESCUE-MBTemp3 #PWR029
+L GND-RESCUE-MBTemp3 #PWR033
 U 1 1 50461F03
 P 2250 4800
-F 0 "#PWR029" H 2250 4800 30  0001 C CNN
+F 0 "#PWR033" H 2250 4800 30  0001 C CNN
 F 1 "GND" H 2250 4730 30  0001 C CNN
 F 2 "" H 2250 4800 60  0001 C CNN
@@
 $EndComp
 $Comp
-L +5V #PWR030
+L +5V #PWR034
 U 1 1 5044CDE6
 P 2400 2600
-F 0 "#PWR030" H 2400 2690 20  0001 C CNN
+F 0 "#PWR034" H 2400 2690 20  0001 C CNN
 F 1 "+5V" H 2400 2690 30  0000 C CNN
 F 2 "" H 2400 2600 60  0001 C CNN
@@
 $EndComp
 $Comp
-L GND-RESCUE-MBTemp3 #PWR031
+L GND-RESCUE-MBTemp3 #PWR035
 U 1 1 5044B39B
 P 1650 2050
-F 0 "#PWR031" H 1650 2050 30  0001 C CNN
+F 0 "#PWR035" H 1650 2050 30  0001 C CNN
 F 1 "GND" H 1650 1980 30  0001 C CNN
 F 2 "" H 1650 2050 60  0001 C CNN
@@
 $EndComp
 $Comp
-L +5V #PWR032
+L +5V #PWR036
 U 1 1 5044AB75
 P 7500 3150
-F 0 "#PWR032" H 7500 3240 20  0001 C CNN
+F 0 "#PWR036" H 7500 3240 20  0001 C CNN
 F 1 "+5V" H 7500 3240 30  0000 C CNN
 F 2 "" H 7500 3150 60  0001 C CNN
@@
 $EndComp
 $Comp
-L GND-RESCUE-MBTemp3 #PWR033
+L GND-RESCUE-MBTemp3 #PWR037
 U 1 1 5044AB66
 P 6750 3950
-F 0 "#PWR033" H 6750 3950 30  0001 C CNN
+F 0 "#PWR037" H 6750 3950 30  0001 C CNN
 F 1 "GND" H 6750 3880 30  0001 C CNN
 F 2 "" H 6750 3950 60  0001 C CNN
@@
 $EndComp
 $Comp
-L +5V #PWR034
+L +5V #PWR038
 U 1 1 503F7C1D
 P 7600 1800
-F 0 "#PWR034" H 7600 1890 20  0001 C CNN
+F 0 "#PWR038" H 7600 1890 20  0001 C CNN
 F 1 "+5V" H 7600 1890 30  0000 C CNN
 F 2 "" H 7600 1800 60  0001 C CNN
@@
 $EndComp
 $Comp
-L GND-RESCUE-MBTemp3 #PWR035
+L GND-RESCUE-MBTemp3 #PWR039
 U 1 1 503F7C1C
 P 7550 2650
-F 0 "#PWR035" H 7550 2650 30  0001 C CNN
+F 0 "#PWR039" H 7550 2650 30  0001 C CNN
 F 1 "GND" H 7550 2580 30  0001 C CNN
 F 2 "" H 7550 2650 60  0001 C CNN
@@
 $EndComp
 $Comp
-L +5V #PWR036
+L +5V #PWR040
 U 1 1 503F7C1A
 P 7800 3500
-F 0 "#PWR036" H 7800 3590 20  0001 C CNN
+F 0 "#PWR040" H 7800 3590 20  0001 C CNN
 F 1 "+5V" H 7800 3590 30  0000 C CNN
 F 2 "" H 7800 3500 60  0001 C CNN
@@
 $EndComp
 $Comp
-L GND-RESCUE-MBTemp3 #PWR037
+L GND-RESCUE-MBTemp3 #PWR041
 U 1 1 503F7C19
 P 7850 4050
-F 0 "#PWR037" H 7850 4050 30  0001 C CNN
+F 0 "#PWR041" H 7850 4050 30  0001 C CNN
 F 1 "GND" H 7850 3980 30  0001 C CNN
 F 2 "" H 7850 4050 60  0001 C CNN
@@
 NoConn ~ 8275 5850
 $Comp
-L GNDREF #PWR038
+L GNDREF #PWR042
 U 1 1 57E1357F
 P 7200 6175
-F 0 "#PWR038" H 7200 5925 50  0001 C CNN
+F 0 "#PWR042" H 7200 5925 50  0001 C CNN
 F 1 "GNDREF" H 7200 6025 50  0000 C CNN
 F 2 "" H 7200 6175 50  0000 C CNN
@@
 $EndComp
 $Comp
-L GNDREF #PWR039
+L GNDREF #PWR043
 U 1 1 57E13893
 P 6950 6175
-F 0 "#PWR039" H 6950 5925 50  0001 C CNN
+F 0 "#PWR043" H 6950 5925 50  0001 C CNN
 F 1 "GNDREF" H 6950 6025 50  0000 C CNN
 F 2 "" H 6950 6175 50  0000 C CNN
@@
 $EndComp
 $Comp
-L GNDREF #PWR040
+L GNDREF #PWR044
 U 1 1 57E138EC
 P 6700 6175
-F 0 "#PWR040" H 6700 5925 50  0001 C CNN
+F 0 "#PWR044" H 6700 5925 50  0001 C CNN
 F 1 "GNDREF" H 6700 6025 50  0000 C CNN
 F 2 "" H 6700 6175 50  0000 C CNN
@@
 Connection ~ 7250 5650
 $Comp
-L GND-RESCUE-MBTemp3 #PWR041
+L GND-RESCUE-MBTemp3 #PWR045
 U 1 1 57E13EF2
 P 8325 5250
-F 0 "#PWR041" H 8325 5250 30  0001 C CNN
+F 0 "#PWR045" H 8325 5250 30  0001 C CNN
 F 1 "GND" H 8325 5180 30  0001 C CNN
 F 2 "" H 8325 5250 60  0001 C CNN
@@
 $EndComp
 $Comp
-L GND-RESCUE-MBTemp3 #PWR042
+L GND-RESCUE-MBTemp3 #PWR046
 U 1 1 57E14221
 P 7125 5450
-F 0 "#PWR042" H 7125 5450 30  0001 C CNN
+F 0 "#PWR046" H 7125 5450 30  0001 C CNN
 F 1 "GND" H 7125 5380 30  0001 C CNN
 F 2 "" H 7125 5450 60  0001 C CNN
@@
 $EndComp
 $Comp
-L +5V #PWR043
+L +5V #PWR047
 U 1 1 57E1430C
 P 7125 4925
-F 0 "#PWR043" H 7125 5015 20  0001 C CNN
+F 0 "#PWR047" H 7125 5015 20  0001 C CNN
 F 1 "+5V" H 7125 5015 30  0000 C CNN
 F 2 "" H 7125 4925 60  0001 C CNN
@@
 Connection ~ 8325 5200
 $Comp
-L +5VP #PWR044
+L +5VP #PWR048
 U 1 1 57E149D2
 P 6700 5800
-F 0 "#PWR044" H 6700 5650 50  0001 C CNN
+F 0 "#PWR048" H 6700 5650 50  0001 C CNN
 F 1 "+5VP" H 6700 5940 50  0000 C CNN
 F 2 "" H 6700 5800 50  0000 C CNN
@@
 Connection ~ 6700 5850
 $Comp
-L GNDREF #PWR045
+L GNDREF #PWR049
 U 1 1 57E156A6
 P 9325 6025
-F 0 "#PWR045" H 9325 5775 50  0001 C CNN
+F 0 "#PWR049" H 9325 5775 50  0001 C CNN
 F 1 "GNDREF" H 9325 5875 50  0000 C CNN
 F 2 "" H 9325 6025 50  0000 C CNN
@@
 $EndComp
 $Comp
-L GNDREF #PWR046
+L GNDREF #PWR050
 U 1 1 57E15705
 P 10300 6025
-F 0 "#PWR046" H 10300 5775 50  0001 C CNN
+F 0 "#PWR050" H 10300 5775 50  0001 C CNN
 F 1 "GNDREF" H 10300 5875 50  0000 C CNN
 F 2 "" H 10300 6025 50  0000 C CNN
@@
 Connection ~ 10300 5800
 $Comp
-L GNDREF #PWR047
+L GNDREF #PWR051
 U 1 1 57E15A80
 P 9675 6025
-F 0 "#PWR047" H 9675 5775 50  0001 C CNN
+F 0 "#PWR051" H 9675 5775 50  0001 C CNN
 F 1 "GNDREF" H 9675 5875 50  0000 C CNN
 F 2 "" H 9675 6025 50  0000 C CNN
@@
 $EndComp
 $Comp
-L GNDREF #PWR048
+L GNDREF #PWR052
 U 1 1 57E15ADF
 P 10650 6025
-F 0 "#PWR048" H 10650 5775 50  0001 C CNN
+F 0 "#PWR052" H 10650 5775 50  0001 C CNN
 F 1 "GNDREF" H 10650 5875 50  0000 C CNN
 F 2 "" H 10650 6025 50  0000 C CNN
@@
 	9675 6025 9675 5750
 $Comp
-L GNDREF #PWR049
+L GNDREF #PWR053
 U 1 1 57E15D2B
 P 9300 2625
-F 0 "#PWR049" H 9300 2375 50  0001 C CNN
+F 0 "#PWR053" H 9300 2375 50  0001 C CNN
 F 1 "GNDREF" H 9300 2475 50  0000 C CNN
 F 2 "" H 9300 2625 50  0000 C CNN
@@
 NoConn ~ 8950 2050
 $Comp
-L +5VP #PWR050
+L +5VP #PWR054
 U 1 1 57E160DA
 P 9100 1800
-F 0 "#PWR050" H 9100 1650 50  0001 C CNN
+F 0 "#PWR054" H 9100 1650 50  0001 C CNN
 F 1 "+5VP" H 9100 1940 50  0000 C CNN
 F 2 "" H 9100 1800 50  0000 C CNN
@@
 	5800 5850 6100 5850
 $Comp
-L GNDREF #PWR051
+L GNDREF #PWR055
 U 1 1 58A48FD4
 P 5800 6125
-F 0 "#PWR051" H 5800 5875 50  0001 C CNN
+F 0 "#PWR055" H 5800 5875 50  0001 C CNN
 F 1 "GNDREF" H 5800 5975 50  0000 C CNN
 F 2 "" H 5800 6125 50  0000 C CNN
@@
 	1    0    0    -1
 $EndComp
+Text GLabel 3500 3150 0    60   Input ~ 0
+I_ENABLE
+Wire Wire Line
+	3500 3150 3600 3150
 $EndSCHEMATC

Commit message: v2.6
Connections:
- net PGC: now reaches P2.3, U7.16 (RB6/PGC)
- net PGD: now reaches P2.5, U7.17 (RB7/PGD)
- net MCLR: now reaches P2.7, U7.18 (MCLR'/VPP)
Changed lines of the file:
@@
 Wire Wire Line
 	3500 3150 3600 3150
+Text Label 7730 3850 0    60   ~ 0
+MCLR
+Text Label 7720 3750 0    60   ~ 0
+PGD
+Text Label 7730 3650 0    60   ~ 0
+PGC
 $EndSCHEMATC
